Commit message: [#134] Add launch files to asimov_simplified and adjust angle limits in urdf

File: robot/rospackages/src/asimov_simplified/urdf/asimov_simplified.urdf (robot description, URDF)
Before this commit: robot asimov_simplified, 8 links, 7 joints
Joints:
- joint distal_joint: limit lower=-1.5708 upper=1.5708 effort=0 velocity=0 -> lower=-3 upper=3 effort=0 velocity=0
- joint finger1_joint: limit lower=-0.01 upper=0 effort=0 velocity=0 -> lower=-0.02 upper=0.005 effort=0 velocity=0
- joint finger2_joint: limit lower=-0.01 upper=0 effort=0 velocity=0 -> lower=-0.02 upper=0.005 effort=0 velocity=0
- joint prox_joint: limit lower=-1.5708 upper=1.5708 effort=0 velocity=0 -> lower=-3 upper=3 effort=0 velocity=0
- joint wrist_flex_joint: limit lower=-1.5708 upper=1.5708 effort=0 velocity=0 -> lower=-3 upper=3 effort=0 velocity=0

Commit message: [#134] Reduce trans_thres to display fine finger motion and adjust translation limits in urdf

File: robot/rospackages/src/asimov_simplified/urdf/asimov_simplified.urdf (robot description, URDF)
Before this commit: robot asimov_simplified, 8 links, 7 joints
Joints:
- joint finger1_joint: limit lower=-0.02 upper=0.005 effort=0 velocity=0 -> lower=-0.02 upper=0.0 effort=0 velocity=0
- joint finger2_joint: limit lower=-0.02 upper=0.005 effort=0 velocity=0 -> lower=-0.02 upper=0.0 effort=0 velocity=0
