Commit message: [#134] Rename actual arm to astro_arm

File: robot/rospackages/src/astro_arm/urdf/astro_arm.urdf (robot description, URDF)
Before this commit: robot SCRB19_MA_000-000-Arm_01.SLDASM, 5 links, 4 joints
Links:
- link base_link: geometry collision mesh filename=package://astro_arm/meshes/base_link.STL; visual mesh filename=package://astro_arm/meshes/base_link.STL
- link distal_link: geometry collision mesh filename=package://astro_arm/meshes/distal_link.STL; visual mesh filename=package://astro_arm/meshes/distal_link.STL
- link proximal_link: geometry collision mesh filename=package://astro_arm/meshes/proximal_link.STL; visual mesh filename=package://astro_arm/meshes/proximal_link.STL
- link upper_base_link: geometry collision mesh filename=package://astro_arm/meshes/upper_base_link.STL; visual mesh filename=package://astro_arm/meshes/upper_base_link.STL
- link wrist: geometry collision mesh filename=package://astro_arm/meshes/wrist.STL; visual mesh filename=package://astro_arm/meshes/wrist.STL

Commit message: [#134] Modify joint names

File: robot/rospackages/src/astro_arm/urdf/astro_arm.urdf (robot description, URDF)
Before this commit: robot astro_arm, 5 links, 4 joints
Joints:
- removed joint motor1
- removed joint motor2
- removed joint motor3
- removed joint motor4
- added joint Elbow Flex: type continuous, parent proximal_link, child distal_link, origin xyz=0.41275 0 0.00160019999999994 rpy=0 0 0, axis 0 0 1
- added joint Shoulder Flex: type continuous, parent upper_base_link, child proximal_link, origin xyz=0 0 0 rpy=1.5708 -1.5708 0, axis 0 0 1
- added joint Shoulder Swivel: type continuous, parent base_link, child upper_base_link, origin xyz=0 -0.002 0.1394 rpy=0 0 0, axis 0 0 1
- added joint Wrist Flex: type continuous, parent distal_link, child wrist, origin xyz=0.4064 0 0 rpy=0 0 0, axis 0 0 1
