Commit message: basic working with stl but some domain issues

File: robot/rospackages/src/arm_ik/urdf/astro_arm.urdf (robot description, URDF)
Before this commit: robot arm_ik, 5 links, 4 joints
Links:
- link base_link: geometry collision mesh filename=package://arm_ik/meshes/base_link.STL; visual mesh filename=package://arm_ik/meshes/base_link.STL

Commit message: Update code to most recent orin repo main branch

File: robot/rospackages/src/arm_ik/urdf/astro_arm.urdf (robot description, URDF)
Before this commit: robot arm_ik, 5 links, 4 joints
Links:
- added link base_footprint
Joints:
- added joint base_joint: type fixed, parent base_footprint, child base_link, origin xyz=0.0 0.0 0.0 rpy=0 0 0
