Commit message: Added worlds. Updated rover model. Updated navigational parameters. Autonomy almost works now, just seems to need functional GPS

File: robot/rospackages/src/beep_autonomy/src/description/rover_description.urdf (robot description, URDF)
Before this commit: robot rover, 4 links, 3 joints
Links:
- added link bogey_b_link; collision box size=${bogey_width} ${base_width+bogey_width} ${bogey_width}; visual box size=${bogey_width} ${base_width+2*bogey_width} ${bogey_width}
- added link gps_link; collision box size=0.1 0.1 0.1; visual box size=0.1 0.1 0.1
- link base_link: geometry collision box size=0.18 ${base_width} 0.08; collision box size=0.68 ${base_width} ${base_height}
- link imu_link: geometry 
Joints:
- added joint bogey_b_joint: type continuous, parent base_link, child bogey_b_link, origin xyz=${-wheel_spacing} 0.0 ${-pivot_zoff} rpy=0.0 0.0 0.0
- added joint gps_joint: type fixed, parent base_link, child gps_link, origin xyz=0 0 0 rpy=0 0 0
- joint imu_joint: origin xyz=0 0 0.01 -> xyz=0.37 0 0.12
- joint lidar_joint: origin xyz=0 0 0.12 rpy=0 0 0 -> xyz=0.37 0 0.12 rpy=0 0 0

Commit message: Modified parameter files. Navigation works

File: robot/rospackages/src/beep_autonomy/src/description/rover_description.urdf (robot description, URDF)
Before this commit: robot rover, 6 links, 5 joints
Joints:
- joint lidar_joint: origin xyz=0.37 0 0.12 rpy=0 0 0 -> xyz=0.37 0 0.2 rpy=0 0 0

Commit message: Simulation updated

File: robot/rospackages/src/beep_autonomy/src/description/rover_description.urdf (robot description, URDF)
Before this commit: robot rover, 6 links, 5 joints
Links:
- added link laser_link, mass 0.125; collision cylinder length=0.055 radius=0.0508; visual cylinder length=0.055 radius=0.0508
Joints:
- added joint laser_joint: type fixed, parent base_link, child laser_link, origin xyz=0.37 0 0.2 rpy=0 0 0

Commit message: Pull latest changes from robotics-orin

File: robot/rospackages/src/beep_autonomy/src/description/rover_description.urdf (robot description, URDF)
Before this commit: robot rover, 8 links, 7 joints
Joints:
- joint zed_joint: child zed_camera_link -> base_footprint; origin xyz=0.4 0 0 -> xyz=-0.4 0 -${(wheel_radius+wheel_height)}; parent base_link -> zed_camera_link

Commit message: in progress to get autonomy working

File: robot/rospackages/src/beep_autonomy/src/description/rover_description.urdf (robot description, URDF)
Before this commit: robot rover, 8 links, 7 joints
Links:
- removed link zed_camera_link
Joints:
- removed joint zed_joint

Commit message: added sim camera

File: robot/rospackages/src/beep_autonomy/src/description/rover_description.urdf (robot description, URDF)
Before this commit: robot rover, 7 links, 6 joints
Links:
- added link camera_link, mass 1e-5; collision box size=${camera_link} ${camera_link} ${camera_link}; visual box size=${camera_link} ${camera_link} ${camera_link}
Joints:
- added joint camera_joint: type fixed, parent laser_link, child camera_link, origin xyz=0.0 0 0.15 rpy=0 0 0

Commit message: copy beep autonomy changes into branch off master

File: robot/rospackages/src/beep_autonomy/src/description/rover_description.urdf (robot description, URDF)
Before this commit: robot rover, 8 links, 7 joints
Links:
- removed link os_imu
- removed link os_lidar
- removed link os_sensor
- removed link zed_camera_link
- added link camera_link, mass 1e-5; collision box size=${camera_link} ${camera_link} ${camera_link}; visual box size=${camera_link} ${camera_link} ${camera_link}
- added link imu_link
- added link laser_link, mass 0.125; collision cylinder length=0.055 radius=0.0508; visual cylinder length=0.055 radius=0.0508
- added link lidar_link, mass 0.125; collision cylinder length=0.055 radius=0.0508; visual cylinder length=0.055 radius=0.0508
Joints:
- removed joint sensor_joint
- removed joint zed_joint
- added joint camera_joint: type fixed, parent laser_link, child camera_link, origin xyz=0.0 0 0.15 rpy=0 0 0
- added joint laser_joint: type fixed, parent base_link, child laser_link, origin xyz=0.37 0 0.2 rpy=0 0 0
- joint bogey_b_joint: type fixed -> continuous
- joint imu_joint: child os_imu -> imu_link; origin xyz=0 0 0.12 -> xyz=0.37 0 0.12
- joint lidar_joint: child os_lidar -> lidar_link; origin xyz=0 0 0.2 rpy=0 0 0 -> xyz=0.37 0 0.2 rpy=0 0 0
